File: led_indicator/schematic.sch (EAGLE design)
At the start: 4 parts

Commit message: update schematics and remove .epf files
Connections:
- net LOGIC_LINE renamed SIGNAL
Changed lines of the file:
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@@
 </segment>
 </net>
-<net name="LOGIC_LINE" class="0">
+<net name="SIGNAL" class="0">
 <segment>
 <pinref part="R1" gate="G$1" pin="1"/>
@@
 <wire x1="33.02" y1="63.5" x2="33.02" y2="60.96" width="0.1524" layer="91"/>
 <wire x1="33.02" y1="60.96" x2="15.24" y2="60.96" width="0.1524" layer="91"/>
-<wire x1="15.24" y1="60.96" x2="-7.62" y2="60.96" width="0.1524" layer="91"/>
-<wire x1="33.02" y1="60.96" x2="55.88" y2="60.96" width="0.1524" layer="91"/>
-<label x="38.1" y="60.96" size="1.778" layer="95"/>
-<label x="-5.08" y="60.96" size="1.778" layer="95"/>
+<wire x1="15.24" y1="60.96" x2="7.62" y2="60.96" width="0.1524" layer="91"/>
+<wire x1="33.02" y1="60.96" x2="40.64" y2="60.96" width="0.1524" layer="91"/>
+<label x="40.64" y="60.96" size="1.778" layer="95" xref="yes"/>
+<label x="7.62" y="60.96" size="1.778" layer="95" rot="MR0" xref="yes"/>
 </segment>
 </net>
