File: RS232_to_serial/max232.sch (EAGLE design)
At the start: 14 parts, among them IC1 MAX232

Commit message: FIXME
Connections:
- net GND: now also R1.2; no longer PWR.C
- net VCC: now also PWR.C; no longer R1.2
Other:
- note added: "v1.1"
Changed lines of the file:
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@@
 <sheet>
 <plain>
+<text x="17.78" y="15.24" size="5.08" layer="97">v1.1</text>
 </plain>
 <instances>
@@
 <attribute name="T2OUT" x="17.78" y="43.18" size="1.778" layer="96" display="name"/>
 </instance>
-<instance part="SUPPLY3" gate="G$1" x="132.08" y="38.1" rot="R270"/>
-<instance part="SUPPLY4" gate="GND" x="99.06" y="17.78" rot="R270"/>
+<instance part="SUPPLY3" gate="G$1" x="99.06" y="17.78" rot="R90"/>
+<instance part="SUPPLY4" gate="GND" x="132.08" y="38.1" rot="R90"/>
 </instances>
 <busses>
@@
 </segment>
 <segment>
-<pinref part="PWR" gate="G$1" pin="C"/>
 <pinref part="SUPPLY4" gate="GND" pin="GND"/>
-<wire x1="104.14" y1="17.78" x2="101.6" y2="17.78" width="0.1524" layer="91"/>
+<pinref part="R1" gate="G$1" pin="2"/>
+<wire x1="129.54" y1="38.1" x2="127" y2="38.1" width="0.1524" layer="91"/>
 </segment>
 </net>
@@
 </segment>
 <segment>
-<pinref part="R1" gate="G$1" pin="2"/>
+<pinref part="PWR" gate="G$1" pin="C"/>
 <pinref part="SUPPLY3" gate="G$1" pin="VCC"/>
-<wire x1="127" y1="38.1" x2="129.54" y2="38.1" width="0.1524" layer="91"/>
+<wire x1="104.14" y1="17.78" x2="101.6" y2="17.78" width="0.1524" layer="91"/>
 </segment>
 </net>
@@
 </sheet>
 </sheets>
+<errors>
+</errors>
 </schematic>
 </drawing>
